File: pcb/test1.brd (EAGLE design)
At the start: 100 x 80 mm, 55 parts, among them IC1 FT232RL, IC2 ACS758ECB-200B-PFF-T, IC3 ACS758ECB-200B-PFF-T, IC4 7805TV, IC5 LM1117, Q1 8mhz, Q2 32khz, U1 STM32F10XRXT6

Commit message: coba board
Parts:
- moved U1 80.1 mm to (40.6, 41.9), flipped to the bottom

Commit message: ready to manufactured and trial
Parts:
- removed JP1: USB_MICROB_PLUGCONN-11752, SparkFun-Connectors:USB-B-MICRO-SMD_V03
- removed JP2: (no value), pinhead:1X04
- removed PAD-V0, PAD-V1: (no value), wirepad:3,81/1,4
- removed PAD33-12, PAD33-5, PAD33-IN: WIREPADSMD2,54-5,08, wirepad:SMD2,54-5,08
- added PAD-33_12, PAD-33_5, PAD-33_IN, PAD-VSS: (no value), wirepad:3,81/1,4
- added TTL: (no value), pinhead:1X04
- added USB: USB_MICROB_PLUGCONN-11752, SparkFun-Connectors:USB-B-MICRO-SMD_V03
- C-33VA, C-5VA, C-PWR1: device resistor:153CLV-1014 -> resistor:E2-5
- D1: value (none) -> 1N4004; device diode:SMC -> diode:DO41-10
- IC4: value 7805TV -> 7805T; device linear:TO220V -> linear:TO220H
- moved BOOT 266.6 mm to (34.4, 54.7)
- moved C-33VB 245.2 mm to (33.9, 26.5), flipped to the bottom
- moved C-33VA 235.5 mm to (33.8, 24.0), turned to 180 degrees
- moved D2 231.3 mm to (34.2, 21.2), flipped to the bottom
- moved R-33B 225.8 mm to (34.0, 15.2), flipped to the bottom, turned to 180 degrees
- moved R-33A 224.1 mm to (34.0, 17.8), flipped to the bottom
- moved IC5 198.5 mm to (32.9, 7.62), turned to 180 degrees
- moved C-5VB 182.6 mm to (21.3, 12.4), flipped to the bottom, turned to 270 degrees
- moved C-5VA 173.3 mm to (19.3, 12.3), turned to 270 degrees
- moved R-VA1 165.7 mm to (50.0, 14.1), flipped to the bottom, turned to 270 degrees
- moved IC3 164.0 mm to (73.8, 12.6), turned to 270 degrees
- moved D1 159.8 mm to (12.8, 5.21), flipped to the bottom
- moved C-PWR2 156.8 mm to (10.5, 9.27), flipped to the bottom, turned to 90 degrees
- moved R-MMC0 153.8 mm to (21.5, 40.9), flipped to the bottom
- moved R-MMC2 152.8 mm to (21.7, 23.7), flipped to the bottom
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Connections:
- removed net N$13: PAD33-12.1
- removed net N$14: PAD33-5.1
- net N$1: now also USB.D-1; no longer JP1.D-1
- net N$12: now also PAD-33_IN.1; no longer PAD33-IN.1
- net N$2: now also USB.D+1; no longer JP1.D+1
- net N$4: now also IC2.IP-, IC2.IP-@10, IC2.IP-@11, IC2.IP-@12, IC2.IP-@13, IC2.IP-@14, IC2.IP-@15, IC2.IP-@16, IC2.IP-@17, IC2.IP-@2, IC2.IP-@3, IC2.IP-@4, IC2.IP-@5, IC2.IP-@6, IC2.IP-@7, IC2.IP-@8, IC2.IP-@9; no longer IC2.IP+, IC2.IP+@10, IC2.IP+@11, IC2.IP+@12, IC2.IP+@13, IC2.IP+@14, IC2.IP+@15, IC2.IP+@16, IC2.IP+@17, IC2.IP+@2, IC2.IP+@3, IC2.IP+@4, IC2.IP+@5, IC2.IP+@6, IC2.IP+@7, IC2.IP+@8, IC2.IP+@9
- net N$5: now also USB.VBUS1; no longer JP1.VBUS1
- net N$7: now also IC3.IP-, IC3.IP-@10, IC3.IP-@11, IC3.IP-@12, IC3.IP-@13, IC3.IP-@14, IC3.IP-@15, IC3.IP-@16, IC3.IP-@17, IC3.IP-@2, IC3.IP-@3, IC3.IP-@4, IC3.IP-@5, IC3.IP-@6, IC3.IP-@7, IC3.IP-@8, IC3.IP-@9; no longer IC3.IP+, IC3.IP+@10, IC3.IP+@11, IC3.IP+@12, IC3.IP+@13, IC3.IP+@14, IC3.IP+@15, IC3.IP+@16, IC3.IP+@17, IC3.IP+@2, IC3.IP+@3, IC3.IP+@4, IC3.IP+@5, IC3.IP+@6, IC3.IP+@7, IC3.IP+@8, IC3.IP+@9
- net RX: now also TTL.2; no longer JP2.2
- net TX: now also TTL.3; no longer JP2.3
- net V12: now also PAD-33_12.1
- net VCC: now also IC1.20, PAD-33_5.1
- net VDD: now also TTL.4; no longer IC1.20, JP2.4
- net VSS: now also PAD-VSS.1, TTL.1, U1.54, USB.GND1, USB.SHIELD1, USB.SHIELD2, USB.SHIELD3; no longer JP1.GND1, JP1.SHIELD1, JP1.SHIELD2, JP1.SHIELD3, JP2.1, PAD-V0.1, PAD-V1.1
Routing:
- net VSS: track 0.00 -> 546.6 mm, vias 0 -> 6
- net VCC: track 0.00 -> 252.8 mm, vias 0 -> 8
- net VDD: track 0.00 -> 251.6 mm, vias 0 -> 10
- net I1: track 0.00 -> 41.0 mm
- net D7: track 0.00 -> 34.2 mm
- net D5: track 0.00 -> 33.6 mm
- net V1: track 0.00 -> 33.5 mm
- net D6: track 0.00 -> 32.6 mm
- net D4: track 0.00 -> 31.8 mm
- net RS: track 0.00 -> 28.0 mm
- net RW: track 0.00 -> 27.1 mm
- net MISO: track 0.00 -> 27.1 mm
- net EN: track 0.00 -> 26.3 mm
- net NSS: track 0.00 -> 25.6 mm, vias 0 -> 2
- net TX: track 0.00 -> 23.9 mm
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- added copper zone on layer 16, net N$21
Other:
- board size 100 x 80 mm -> 87 x 78.2 mm

Commit message: revisi layout
Routing:
- net VCC: track 252.8 -> 264.0 mm, vias 8 -> 10
Changed lines of the file:
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@@
 <layer number="21" name="tPlace" color="7" fill="1" visible="yes" active="yes"/>
 <layer number="22" name="bPlace" color="7" fill="1" visible="yes" active="yes"/>
-<layer number="23" name="tOrigins" color="15" fill="1" visible="yes" active="yes"/>
-<layer number="24" name="bOrigins" color="15" fill="1" visible="yes" active="yes"/>
-<layer number="25" name="tNames" color="7" fill="1" visible="yes" active="yes"/>
-<layer number="26" name="bNames" color="7" fill="1" visible="yes" active="yes"/>
+<layer number="23" name="tOrigins" color="15" fill="1" visible="no" active="yes"/>
+<layer number="24" name="bOrigins" color="15" fill="1" visible="no" active="yes"/>
+<layer number="25" name="tNames" color="7" fill="1" visible="no" active="yes"/>
+<layer number="26" name="bNames" color="7" fill="1" visible="no" active="yes"/>
 <layer number="27" name="tValues" color="7" fill="1" visible="no" active="yes"/>
 <layer number="28" name="bValues" color="7" fill="1" visible="no" active="yes"/>
@@
 <wire x1="17.653" y1="70.358" x2="17.653" y2="71.503" width="0.4064" layer="16"/>
 <wire x1="17.653" y1="71.503" x2="17.657" y2="71.507" width="0.4064" layer="16"/>
-<wire x1="52.26" y1="37.597" x2="53.335" y2="37.597" width="0.3048" layer="16"/>
-<wire x1="53.335" y1="37.597" x2="55.499" y2="35.433" width="0.3048" layer="16"/>
-<wire x1="55.499" y1="35.433" x2="55.499" y2="31.75" width="0.3048" layer="16"/>
 <via x="40.767" y="28.194" extent="1-16" drill="0.9" shape="octagon"/>
 <wire x1="40.767" y1="28.194" x2="40.767" y2="11.684" width="0.3048" layer="16"/>
@@
 <wire x1="40.767" y1="28.194" x2="45.212" y2="28.194" width="0.3048" layer="1"/>
 <via x="45.212" y="28.194" extent="1-16" drill="0.9" shape="octagon"/>
-<wire x1="45.212" y1="28.194" x2="51.943" y2="28.194" width="0.3048" layer="16"/>
+<wire x1="45.212" y1="28.194" x2="49.022" y2="28.194" width="0.3048" layer="16"/>
+<wire x1="49.022" y1="28.194" x2="51.943" y2="28.194" width="0.3048" layer="16"/>
 <wire x1="51.943" y1="28.194" x2="55.499" y2="31.75" width="0.3048" layer="16"/>
-<wire x1="55.499" y1="35.433" x2="55.499" y2="36.195" width="0.3048" layer="16"/>
-<wire x1="55.499" y1="36.195" x2="56.261" y2="36.957" width="0.3048" layer="16"/>
-<via x="56.261" y="36.957" extent="1-16" drill="0.9" shape="octagon"/>
-<wire x1="56.261" y1="36.957" x2="56.261" y2="72.39" width="0.3048" layer="1"/>
 <via x="56.261" y="72.39" extent="1-16" drill="0.9" shape="octagon"/>
 <wire x1="56.261" y1="72.39" x2="56.261" y2="72.644" width="0.3048" layer="16"/>
@@
 <wire x1="47.244" y1="75.819" x2="53.086" y2="75.819" width="0.3048" layer="16"/>
 <wire x1="53.086" y1="75.819" x2="56.261" y2="72.644" width="0.3048" layer="16"/>
+<wire x1="56.261" y1="72.39" x2="56.261" y2="63.881" width="0.4064" layer="1"/>
+<via x="56.261" y="63.881" extent="1-16" drill="0.9" shape="octagon"/>
+<wire x1="56.261" y1="63.881" x2="56.261" y2="46.228" width="0.4064" layer="16"/>
+<wire x1="56.261" y1="46.228" x2="51.054" y2="41.021" width="0.4064" layer="16"/>
+<wire x1="51.054" y1="41.021" x2="49.149" y2="41.021" width="0.4064" layer="16"/>
+<wire x1="49.149" y1="41.021" x2="49.022" y2="40.894" width="0.4064" layer="16"/>
+<via x="49.022" y="40.894" extent="1-16" drill="0.9" shape="octagon"/>
+<wire x1="49.022" y1="40.894" x2="49.022" y2="28.702" width="0.4064" layer="1"/>
+<via x="49.022" y="28.702" extent="1-16" drill="0.9" shape="octagon"/>
+<wire x1="49.022" y1="28.702" x2="49.022" y2="28.194" width="0.4064" layer="16"/>
+<wire x1="52.26" y1="37.597" x2="53.589" y2="37.597" width="0.4064" layer="16"/>
+<wire x1="53.589" y1="37.597" x2="55.499" y2="35.687" width="0.4064" layer="16"/>
+<wire x1="55.499" y1="35.687" x2="55.499" y2="31.75" width="0.4064" layer="16"/>
 </signal>
 <signal name="N$4">

Commit message: Calibrated & Ready to test
Parts:
- moved L-RUN 0.63 mm to (13.2, 46.9)
- moved R-RUN 0.63 mm to (8.26, 46.9)
Routing:
- net VDD: track 251.6 -> 252.2 mm
Changed lines of the file:
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@@
 <layer number="21" name="tPlace" color="7" fill="1" visible="yes" active="yes"/>
 <layer number="22" name="bPlace" color="7" fill="1" visible="yes" active="yes"/>
-<layer number="23" name="tOrigins" color="15" fill="1" visible="no" active="yes"/>
-<layer number="24" name="bOrigins" color="15" fill="1" visible="no" active="yes"/>
+<layer number="23" name="tOrigins" color="15" fill="1" visible="yes" active="yes"/>
+<layer number="24" name="bOrigins" color="15" fill="1" visible="yes" active="yes"/>
 <layer number="25" name="tNames" color="7" fill="1" visible="no" active="yes"/>
 <layer number="26" name="bNames" color="7" fill="1" visible="no" active="yes"/>
@@
 <element name="L-PWR" library="led" package="SML1206" value="" x="13.208" y="49.276" rot="MR0"/>
 <element name="R-PWR" library="resistor" package="R1206" value="330" x="8.255" y="49.403" rot="MR0"/>
-<element name="R-RUN" library="resistor" package="R1206" value="330" x="8.255" y="47.498" rot="MR0"/>
-<element name="L-RUN" library="led" package="SML1206" value="" x="13.208" y="47.498" rot="MR0"/>
+<element name="R-RUN" library="resistor" package="R1206" value="330" x="8.255" y="46.863" rot="MR0"/>
+<element name="L-RUN" library="led" package="SML1206" value="" x="13.208" y="46.863" rot="MR0"/>
 <element name="DIS1" library="display-lcd" package="TUXGR_16X2_R2" value="TUXGR_16X2_R2" x="47.117" y="56.007">
 <attribute name="OC_NEWARK" value="unknown" x="100.457" y="36.957" size="1.778" layer="27" display="off"/>
@@
 <wire x1="25.15" y1="41.144" x2="24.003" y2="42.291" width="0.3048" layer="16"/>
 <wire x1="24.003" y1="42.291" x2="24.003" y2="44.831" width="0.3048" layer="16"/>
-<wire x1="24.003" y1="44.831" x2="21.717" y2="47.117" width="0.3048" layer="16"/>
-<wire x1="21.717" y1="47.117" x2="15.339" y2="47.117" width="0.3048" layer="16"/>
-<wire x1="15.339" y1="47.117" x2="14.958" y2="47.498" width="0.3048" layer="16"/>
+<wire x1="24.003" y1="44.831" x2="21.59" y2="47.244" width="0.3048" layer="16"/>
+<wire x1="14.958" y1="46.863" x2="16.383" y2="46.863" width="0.3048" layer="16"/>
+<wire x1="16.383" y1="46.863" x2="16.764" y2="47.244" width="0.3048" layer="16"/>
+<wire x1="16.764" y1="47.244" x2="21.59" y2="47.244" width="0.3048" layer="16"/>
 </signal>
 <signal name="VDD">
@@
 <contactref element="U1" pad="7"/>
 <contactref element="BOOT" pad="3"/>
-<wire x1="6.833" y1="47.498" x2="6.833" y2="49.403" width="0.3048" layer="16"/>
 <wire x1="32.893" y1="11.43" x2="32.893" y2="11.811" width="0.8128" layer="16"/>
 <wire x1="32.893" y1="11.811" x2="30.607" y2="14.097" width="0.8128" layer="16"/>
@@
 <wire x1="40.005" y1="59.69" x2="36.957" y2="56.642" width="0.3048" layer="16"/>
 <wire x1="36.957" y1="56.642" x2="36.957" y2="54.737" width="0.3048" layer="16"/>
+<wire x1="6.833" y1="49.403" x2="6.833" y2="46.863" width="0.3048" layer="16"/>
 </signal>
 <signal name="VSS">
@@
 <contactref element="R-RUN" pad="1"/>
 <contactref element="L-RUN" pad="A"/>
-<wire x1="11.458" y1="47.498" x2="9.677" y2="47.498" width="0.3048" layer="16"/>
+<wire x1="11.458" y1="46.863" x2="9.677" y2="46.863" width="0.3048" layer="16"/>
 </signal>
 <signal name="N$8">
